File: H743_LCD_dev.kicad_pcb (KiCad board)
At the start: 6 copper layers, 76 x 78 mm, 134 parts, among them J1 Micro_SD_Card_Det_Hirose_DM3AT, J2 TFT_LCD, J4 USB-C, J5 I2C-STEMMA-QT, J6 BAT, J7 swd, J8 SPKR, J9 UART, SW1 SW_Push, SW2 SW_Push, SW3 SW_Push, SW4 SW_Push, U1 MT25Q, U2 IS42S16160J-7TL, U4 STM32H723ZGTx, U5 TPS61169, U6 MAX98357AETE_, U7 CAT24C128, U8 TLV75733PDBV, U9 W25Q128JVS, Y1 25MHz, Y2 32.768KHz

Commit message: Finished. 1st version, ordered 1st batch
Parts:
- added C50: 1u, Capacitor_SMD:C_0603_1608Metric, F.Cu at (142.5, 119.2)
- added G***: LOGO, chroma_pixel:chroma_pixel, F.Cu at (144.5, 64.9)
- added kibuzzard-66458F69: G***, kibuzzard-66458F69, F.Cu at (172.0, 51.7)
- added kibuzzard-66458F9C: G***, kibuzzard-66458F9C, F.Cu at (165.0, 51.7)
- D7: footprint Package_TO_SOT_SMD:SOT-323_SC-70 -> Package_TO_SOT_SMD:SOT-23
- L2: footprint Inductor_SMD:L_1210_3225Metric -> Inductor_SMD:L_Changjiang_FNR5012S
- R16: value NC -> 100K
- moved JP4 3.08 mm to (131.4, 59.8)
- moved C49 3.08 mm to (122.6, 59.3)
- moved C48 3.08 mm to (128.3, 58.4)
- moved R25 3.08 mm to (121.3, 59.2)
- moved R29 3.08 mm to (128.3, 59.7)
- moved U5 3.08 mm to (125.0, 59.1)
- moved R26 3.08 mm to (119.5, 59.7)
- moved R27 3.08 mm to (119.5, 58.5)
- moved R28 3.08 mm to (119.5, 57.2)
- moved kibuzzard-6642BE6C 2.29 mm to (141.2, 116.5)
- moved L2 1.71 mm to (125.0, 54.7)
- moved kibuzzard-6642BE54 0.51 mm to (133.8, 116.5)
Connections:
- U4 pad 116: /MCU/PD2 -> /LCD/LCD_B7
- U4 pad 140: /LCD/LCD_B7 -> /MCU/PB9
Routing:
- net /LCD/LCD_B7: track 47.7 -> 61.9 mm
- net Net-(D8-A): track 5.49 -> 8.73 mm
- net /LCD/LCD_BLK: track 42.9 -> 46.0 mm
- net /MCU/NOR_D3: track 27.9 -> 30.9 mm
- net /MCU/NOR_D0: track 27.9 -> 30.9 mm
- net /MCU/NOR_D1: track 27.9 -> 30.9 mm
- net /MCU/NOR_D2: track 27.9 -> 30.9 mm
- net Net-(JP2-B): track 5.36 -> 2.76 mm
- net /LCD/LED_K: track 24.8 -> 27.1 mm
- net /MCU/PG15: track 51.4 -> 53.6 mm
- net Net-(JP1-B): track 7.34 -> 5.23 mm
- net GND: track 159.6 -> 161.4 mm
- net /MCU/PC5: track 46.2 -> 47.6 mm
- net /MCU/PG4: track 51.4 -> 52.6 mm
- net /MCU/PC4: track 26.7 -> 27.7 mm
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- added copper zone on F.Cu, net +3V3
Other:
- outline, holes or cut-outs redrawn
- board text added: "Backlight"
- board text added: "PWM_BL"
- board text added: "current"
- board text removed: "Backlight current"
