File: H743_LCD_dev.kicad_sch (KiCad schematic)
At the start: 4 parts

Commit message: Finished. 1st version, ordered 1st batch
Changed lines of the file:
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@@
+		)
+	)
+	(polyline
+		(pts
+			(xy 186.055 64.77) (xy 202.565 64.77)
+		)
+		(stroke
+			(width 0)
+			(type default)
 		)
 	)
@@
 		)
 		(stroke
-			(width 0)
-			(type default)
-		)
-	)
-	(polyline
-		(pts
-			(xy 180.34 64.77) (xy 202.565 64.77)
-		)
-		(stroke
