File: MAX98357.kicad_sch (KiCad schematic)
At the start: 6 parts, among them J8 SPKR, U6 MAX98357AETE_

Commit message: Looks like FPC should be changed to XF2M-4015-1A
Parts:
- U6: JLCPCB Part # (none) -> C910544
Changed lines of the file:
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@@
+			)
+		)
+		(property "JLCPCB Part #" ""
+			(at 67.31 96.52 0)
+			(effects
+				(font
+					(size 1.27 1.27)
+				)
+				(hide yes)
 			)
 		)
@@
 			)
 		)
+		(property "JLCPCB Part #" ""
+			(at 67.31 88.9 0)
+			(effects
+				(font
+					(size 1.27 1.27)
+				)
+				(hide yes)
+			)
+		)
 		(pin "1"
 		)
@@
 			)
 		)
+		(property "JLCPCB Part #" "C910544"
+			(at 140.97 90.17 0)
+			(effects
+				(font
+					(size 1.27 1.27)
+				)
+				(hide yes)
+			)
+		)
 		(pin "11"
 		)
@@
 			)
 		)
+		(property "JLCPCB Part #" ""
+			(at 111.76 95.25 0)
+			(effects
+				(font
+					(size 1.27 1.27)
+				)
+				(hide yes)
+			)
+		)
 		(pin "1"
 		)
@@
 			)
 		)
+		(property "JLCPCB Part #" ""
+			(at 177.8 77.47 0)
+			(effects
+				(font
+					(size 1.27 1.27)
+				)
+				(hide yes)
+			)
+		)
 		(pin "1"
 		)
@@
 			(at 219.71 85.09 0)
 			(effects
+				(font
+					(size 1.27 1.27)
+				)
+				(hide yes)
+			)
+		)
+		(property "JLCPCB Part #" ""
+			(at 219.71 85.09 0)
+			(effects

Commit message: Changed the FPC footprint and uart, added RTC battery connector
Parts:
- J8: JLCPCB Part # (none) -> C7419891

Commit message: Added UART esd
Parts:
- C23: JLCPCB Part # (none) -> C96446
- R14: JLCPCB Part # (none) -> C26083
Changed lines of the file:
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@@
 			)
 		)
-		(property "JLCPCB Part #" ""
+		(property "JLCPCB Part #" "C26083"
 			(at 111.76 95.25 0)
 			(effects
@@
 			)
 		)
-		(property "JLCPCB Part #" ""
+		(property "JLCPCB Part #" "C96446"
 			(at 177.8 77.47 0)
 			(effects

Commit message: Finished. 1st version, ordered 1st batch
Parts:
- R15: now not fitted; now left out of the parts list
- R16: value NC -> 100K; JLCPCB Part # (none) -> C25741
Other:
- note added: "gain=15"
Changed lines of the file:
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@@
+		)
+	)
+	(text "gain=15"
+		(exclude_from_sim no)
+		(at 79.502 96.52 0)
+		(effects
+			(font
+				(size 1.27 1.27)
+			)
 		)
 	)
@@
 			)
 		)
-		(property "Value" "NC"
+		(property "Value" "100K"
 			(at 69.85 97.7899 0)
 			(effects
@@
 			)
 		)
-		(property "JLCPCB Part #" ""
+		(property "JLCPCB Part #" "C25741"
 			(at 67.31 96.52 0)
 			(effects
@@
 		(unit 1)
 		(exclude_from_sim no)
-		(in_bom yes)
+		(in_bom no)
 		(on_board yes)
-		(dnp no)
+		(dnp yes)
 		(fields_autoplaced yes)
 		(property "Reference" "R15"
