File: STM32H743IIK6.kicad_sch (KiCad schematic)
At the start: 57 parts, among them J4 USB-C, J6 BAT, SW1 SW_Push, SW2 SW_Push, SW3 SW_Push, SW4 SW_Push, U4 STM32H723ZGTx, U8 TLV75733PDBV, Y1 25MHz, Y2 32.768KHz

Commit message: All clear (need verification), need add capacitor next to I2C conn, verify I2S gain
Connections:
- net SHIELD: now reaches C43.1, J4.S1 (SHIELD), R13.1
Other:
- moved on the sheet: R13

Commit message: Finished. 1st version, ordered 1st batch
Parts:
- D7: footprint Package_TO_SOT_SMD:SOT-323_SC-70 -> Package_TO_SOT_SMD:SOT-23
Connections:
- net PD2 is gone; now on net LTDC_B7: U4.116 (PD2)
- net LTDC_B7: no longer U4.140 (PB9)
- new net PB9: U4.140 (PB9)
Other:
- note added: "Verified"
